Commit message: urdf: single clean cylinder wheel collider (was 2 cylinders + mesh hull -> no grip)

File: leorover_isaac/assets/leo_rover/source/leo_robot_1_ros2_shared.urdf (robot description, URDF)
Before this commit: robot leo_robot_1_ros2_shared, 7 links, 6 joints
Links:
- link wheel_FL_link: geometry collision cylinder length=0.07 radius=0.0625; visual mesh filename=WheelA.dae
- link wheel_FR_link: geometry collision cylinder length=0.07 radius=0.0625; visual mesh filename=WheelB.dae
- link wheel_RL_link: geometry collision cylinder length=0.07 radius=0.0625; visual mesh filename=WheelA.dae
- link wheel_RR_link: geometry collision cylinder length=0.07 radius=0.0625; visual mesh filename=WheelB.dae

Commit message: urdf: sphere wheel colliders (cylinder gets faceted to a prism in PhysX -> no roll)

File: leorover_isaac/assets/leo_rover/source/leo_robot_1_ros2_shared.urdf (robot description, URDF)
Before this commit: robot leo_robot_1_ros2_shared, 7 links, 6 joints
Links:
- link wheel_FL_link: geometry collision sphere radius=0.0625; visual mesh filename=WheelA.dae
- link wheel_FR_link: geometry collision sphere radius=0.0625; visual mesh filename=WheelB.dae
- link wheel_RL_link: geometry collision sphere radius=0.0625; visual mesh filename=WheelA.dae
- link wheel_RR_link: geometry collision sphere radius=0.0625; visual mesh filename=WheelB.dae
