Commit message: wheels: restore PyBullet cylinder collider (2 coaxial cyl + outline) over the sphere; keep PhysX smooth cylinder-vs-trimesh collision

File: leorover_isaac/assets/leo_rover/source/leo_robot_1_ros2_shared.urdf (robot description, URDF)
Before this commit: robot leo_robot_1_ros2_shared, 7 links, 6 joints
Links:
- link wheel_FL_link: geometry collision cylinder length=0.04 radius=0.0625; collision cylinder length=0.07 radius=0.057
- link wheel_FR_link: geometry collision cylinder length=0.04 radius=0.0625; collision cylinder length=0.07 radius=0.057
- link wheel_RL_link: geometry collision cylinder length=0.04 radius=0.0625; collision cylinder length=0.07 radius=0.057
- link wheel_RR_link: geometry collision cylinder length=0.04 radius=0.0625; collision cylinder length=0.07 radius=0.057
